Commit message: updated robot models

File: amr_description/urdf/AMR_Platform.urdf (robot description, URDF)
Before this commit: robot AMR_Platform, 8 links, 7 joints
Links:
- link main_body: geometry collision mesh filename=package://amr_description/meshes/AMR_Platform.STL; visual mesh filename=package://amr_description/meshes/AMR_Platform.STL

File: amr_description/urdf/LD250.urdf (robot description, URDF)
Before this commit: robot LD90, 2 links, 1 joints
Links:
- link main_body: geometry collision mesh filename=package://amr_description/meshes/LD250.obj; visual mesh filename=package://amr_description/meshes/LD250.obj

File: amr_description/urdf/LD90.urdf (robot description, URDF)
Before this commit: robot LD90, 2 links, 1 joints
Links:
- link main_body: geometry collision mesh filename=package://amr_description/meshes/LD90.obj; visual mesh filename=package://amr_description/meshes/LD90.obj
