Commit message: fixed missing laser interface error

File: amr_description/urdf/LD250.urdf (robot description, URDF)
Before this commit: robot LD250, 3 links, 2 joints
Links:
- removed link main_body
- added link amr_base, mass 4.07; collision mesh filename=package://amr_description/meshes/LD250.obj; visual mesh filename=package://amr_description/meshes/LD250.obj
- added link laser_frame_low
Joints:
- removed joint main_body_to_base
- added joint amr_base_to_base_link: type fixed, parent base_link, child amr_base, origin xyz=0 0 0
- added joint base_link_to_laser_frame_low: type fixed, parent base_link, child laser_frame_low, origin xyz=0.40 0 0.060
- joint base_link_to_laser_frame: origin xyz=0.45 0 0.195 -> xyz=0.40 0 0.190

File: amr_description/xacro/ld250.urdf.xacro (robot description, xacro)
@@ -4,6 +4,7 @@
     Updated to match LD250.urdf:
     - Adds laser_frame link
-    - Adds base_link_to_laser_frame fixed joint at xyz="0.45 0 0.195"
-    - Keeps main_body mesh, inertial, and fixed joints
+    - Adds laser_frame_low link
+    - Adds base_link_to_laser_frame fixed joint at xyz="0.40 0 0.190"
+    - Keeps amr_base mesh, inertial, and fixed joints
   -->
   <xacro:macro name="ld250" params="prefix:='' parent:='' xyz:='0 0 0' rpy:='0 0 0' mesh_pkg:='amr_description'">
@@ -16,5 +17,5 @@
     </link>
     <!-- Main body with mesh -->
-    <link name="${prefix}main_body">
+    <link name="${prefix}amr_base">
       <visual>
         <origin rpy="0 0 3.141582654" xyz="0 0 0"/>
@@ -35,8 +36,8 @@
       </inertial>
     </link>
-    <!-- Base to main body fixed joint -->
-    <joint name="${prefix}main_body_to_base" type="fixed">
+    <!-- Base link to main body fixed joint -->
+    <joint name="${prefix}amr_base_to_base_link" type="fixed">
       <parent link="${prefix}base_link"/>
-      <child link="${prefix}main_body"/>
+      <child link="${prefix}amr_base"/>
       <origin xyz="0 0 0"/>
     </joint>
@@ -48,5 +49,13 @@
       <parent link="${prefix}base_link"/>
       <child link="${prefix}laser_frame"/>
-      <origin xyz="0.45 0 0.195"/>
+      <origin xyz="0.40 0 0.190"/>
+    </joint>
+        <!-- Low front laser frame -->
+    <link name="${prefix}laser_frame_low">
+    </link>
+    <joint name="${prefix}base_link_to_laser_frame_low" type="fixed">
+      <parent link="${prefix}base_link"/>
+      <child link="${prefix}laser_frame_low"/>
+      <origin xyz="0.40 0 0.060"/>
     </joint>
     <!-- Optional mounting to an external parent -->
@@ -59,11 +68,15 @@
     </xacro:if>
     <!--
-      Dimensions (from LD250.urdf comments):
-      - length: 950 mm
-      - width: 696 mm
-      - laser glass offset front: 20 mm
-      - laser glass offset back: 120 mm
-      - laser glass bottom height: 180 mm
-      - laser glass top height: 210 mm
+      Dimensions (from https://files.omron.eu/downloads/latest/datasheet/en/i828_ld-series_mobile_robot_datasheet_en.pdf?v=2):
+      - length: 970 mm
+      - width: 720 mm
+      - base height: 380 mm
+      - laser glass center height: 190 mm
+      Dimensions roughly measured
+      - laser glass offset front: 35 mm
+      - laser glass offset back: 135 mm
+      - lower laser glass center height: 60 mm
+      Calaculated from the above dimensions:
+      - laser center from the middle of the robot: (970/2 - 135 + (135-35)/2) mm = 400 mm
     -->
   </xacro:macro>
